Commit message: Fixed URDF for SUPleft arm 3 joints

File: URDF/ArmsnHands.SLDASM/urdf/ArmsnHands.SLDASM.urdf (robot description, URDF)
Before this commit: robot ArmsnHands.SLDASM, 4 links, 3 joints
Joints:
- joint elbow_joint: axis 0 0 0 -> 0 0 1; type fixed -> revolute
- joint foreamr_roll_joint: axis 0 0 0 -> 1 0 0; type fixed -> revolute
- joint forearm_updown_joint: axis 0 0 0 -> 0 0 1; origin xyz=0.00051304 0.4837 -0.00034787 rpy=-1.5708 0 1.5708 -> xyz=0.00051304 0.2537 -0.00034787 rpy=-1.5708 0 1.5708; type fixed -> revolute
