Commit message: add 3 dof Sup arm

File: URDF/ArmsnHandsR.SLDASM/urdf/ArmsnHandsR.SLDASM.urdf (robot description, URDF)
Before this commit: robot ArmsnHandsR.SLDASM, 4 links, 3 joints
Joints:
- joint elbow_joint: axis 0 0 0 -> 0 0 1; origin xyz=0.205 -0.0015189 5.7522E-05 rpy=-1.6086 0 0 -> xyz=-0.205 -0.0015189 5.7522E-05 rpy=-1.6086 0 0
- joint foreamr_roll_joint: axis 0 0 0 -> 1 0 0; origin xyz=0 0 0 rpy=0 0 0 -> xyz=0 -0.01309 0 rpy=0 0 0
- joint forearm_updown_joint: axis 0 0 0 -> 0 0 1; origin xyz=0.00051304 0.4837 -0.00034787 rpy=-1.5708 0 1.5708 -> xyz=0.00051304 0.2537 -0.00034787 rpy=-1.5708 0 1.5708
